File: Contrib/docvolt/adapter/schematic.kicad_sch (KiCad schematic)
At the start: 37 parts, among them J1 Audio, J2 NES Controller, J3 Conn_01x06_Socket, J5 VGA, U1 TXB0104D, U2 Tang Nano 9K, U3 TXB0104D, U4 TXB0104D

Commit message: FPGA implementation
Connections:
- net DATA is gone; now on net SER_DATA: D1.1 (K), J2.2, R18.1
- net HSYNC is gone; now on net SER_PULSE: J2.4, J5.13, U3.12 (B2)
- net VSYNC is gone; now on net SER_LATCH: J2.3, J5.14, U3.13 (B1)
Changed lines of the file:
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@@
 	)
 	(junction
+		(at 232.41 63.5)
+		(diameter 0)
+		(color 0 0 0 0)
+	)
+	(junction
 		(at 78.74 78.74)
 		(diameter 0)
@@
 		(color 0 0 0 0)
 	)
+	(junction
+		(at 59.69 137.16)
+		(diameter 0)
+		(color 0 0 0 0)
+	)
 	(no_connect
 		(at 243.84 118.11)
@@
 	(wire
 		(pts
+			(xy 44.45 137.16) (xy 59.69 137.16)
+		)
+		(stroke
+			(width 0)
+			(type default)
+		)
+	)
+	(wire
+		(pts
 			(xy 102.87 90.17) (xy 96.52 90.17)
 		)
@@
 	(wire
 		(pts
+			(xy 59.69 137.16) (xy 76.2 137.16)
+		)
+		(stroke
+			(width 0)
+			(type default)
+		)
+	)
+	(wire
+		(pts
 			(xy 190.5 73.66) (xy 186.69 73.66)
 		)
@@
 	(wire
 		(pts
+			(xy 59.69 142.24) (xy 62.23 142.24)
+		)
+		(stroke
+			(width 0)
+			(type default)
+		)
+	)
+	(wire
+		(pts
 			(xy 53.34 73.66) (xy 53.34 55.88)
 		)
@@
 	(wire
 		(pts
+			(xy 59.69 147.32) (xy 63.5 147.32)
+		)
+		(stroke
+			(width 0)
+			(type default)
+		)
+	)
+	(wire
+		(pts
 			(xy 234.95 83.82) (xy 229.87 83.82)
 		)
@@
 	(wire
 		(pts
-			(xy 59.69 142.24) (xy 69.85 142.24)
-		)
-		(stroke
-			(width 0)
-			(type default)
-		)
-	)
-	(wire
-		(pts
-			(xy 59.69 147.32) (xy 69.85 147.32)
-		)
-		(stroke
-			(width 0)
-			(type default)
-		)
-	)
-	(wire
-		(pts
 			(xy 95.25 90.17) (xy 95.25 95.25)
 		)
@@
 	(wire
 		(pts
+			(xy 232.41 63.5) (xy 240.03 63.5)
+		)
+		(stroke
+			(width 0)
+			(type default)
+		)
+	)
+	(wire
+		(pts
 			(xy 201.93 73.66) (xy 201.93 88.9)
 		)
@@
 	(wire
 		(pts
-			(xy 59.69 137.16) (xy 76.2 137.16)
-		)
-		(stroke
-			(width 0)
-			(type default)
-		)
-	)
-	(wire
-		(pts
 			(xy 186.69 115.57) (xy 190.5 115.57)
 		)
@@
 		)
 	)
-	(label "DATA"
-		(at 59.69 137.16 0)
+	(label "Red"
+		(at 201.93 113.03 0)
 		(fields_autoplaced yes)
 		(effects
@@
 		)
 	)
-	(label "VSYNC"
-		(at 234.95 58.42 180)
+	(label "PULSE"
+		(at 166.37 63.5 180)
 		(fields_autoplaced yes)
 		(effects
@@
 		)
 	)
-	(label "Red"
-		(at 201.93 113.03 0)
+	(label "Blue"
+		(at 201.93 68.58 0)
 		(fields_autoplaced yes)
 		(effects
@@
 		)
 	)
-	(label "VSYNC"
-		(at 69.85 142.24 180)
+	(label "Green"
+		(at 201.93 100.33 0)
 		(fields_autoplaced yes)
 		(effects
@@
 				(size 1.27 1.27)
 			)
-			(justify right bottom)
+			(justify left bottom)
 		)
 	)
-	(label "PULSE"
-		(at 166.37 63.5 180)
+	(global_label "SER_DATA"
+		(shape input)
+		(at 243.84 151.13 180)
 		(fields_autoplaced yes)
 		(effects
@@
 				(size 1.27 1.27)
 			)
-			(justify right bottom)
+			(justify right)
 		)
-	)
-	(label "Blue"
-		(at 201.93 68.58 0)
-		(fields_autoplaced yes)
-		(effects
-			(font
-				(size 1.27 1.27)
+		(property "Intersheetrefs" "${INTERSHEET_REFS}"
+			(at 231.8439 151.13 0)
+			(effects
+				(font
+					(size 1.27 1.27)
+				)
+				(justify right)
+				(hide yes)
 			)
-			(justify left bottom)
 		)
 	)
-	(label "HSYNC"
-		(at 232.41 63.5 180)
+	(global_label "SER_LATCH"
+		(shape input)
+		(at 234.95 58.42 0)
 		(fields_autoplaced yes)
 		(effects
@@
 				(size 1.27 1.27)
 			)
-			(justify right bottom)
+			(justify left)
+		)
+		(property "Intersheetrefs" "${INTERSHEET_REFS}"
+			(at 248.2161 58.42 0)
+			(effects
+				(font
+					(size 1.27 1.27)
+				)
+				(justify left)
+				(hide yes)
+			)
 		)
 	)
-	(label "HSYNC"
-		(at 69.85 147.32 180)
+	(global_label "SER_PULSE"
+		(shape input)
+		(at 240.03 63.5 0)
 		(fields_autoplaced yes)
 		(effects
@@
 				(size 1.27 1.27)
 			)
-			(justify right bottom)
+			(justify left)
+		)
+		(property "Intersheetrefs" "${INTERSHEET_REFS}"
+			(at 253.5984 63.5 0)
+			(effects
+				(font
+					(size 1.27 1.27)
+				)
+				(justify left)
+				(hide yes)
+			)
 		)
 	)
-	(label "Green"
-		(at 201.93 100.33 0)
+	(global_label "SER_LATCH"
+		(shape input)
+		(at 62.23 142.24 0)
 		(fields_autoplaced yes)
 		(effects
@@
 				(size 1.27 1.27)
 			)
-			(justify left bottom)
+			(justify left)
+		)
+		(property "Intersheetrefs" "${INTERSHEET_REFS}"
+			(at 75.4961 142.24 0)
+			(effects
+				(font
+					(size 1.27 1.27)
+				)
+				(justify left)
+				(hide yes)
+			)
 		)
 	)
 	(global_label "SER_DATA"
 		(shape input)
-		(at 243.84 151.13 180)
+		(at 44.45 137.16 180)
 		(fields_autoplaced yes)
 		(effects
@@
 		)
 		(property "Intersheetrefs" "${INTERSHEET_REFS}"
-			(at 231.8439 151.13 0)
+			(at 32.4539 137.16 0)
 			(effects
 				(font
@@
 		)
 	)
+	(global_label "SER_PULSE"
+		(shape input)
+		(at 63.5 147.32 0)
+		(fields_autoplaced yes)
+		(effects
+			(font
+				(size 1.27 1.27)
+			)
+			(justify left)
+		)
+		(property "Intersheetrefs" "${INTERSHEET_REFS}"
+			(at 77.0684 147.32 0)
+			(effects
+				(font
+					(size 1.27 1.27)
+				)
+				(justify left)
+				(hide yes)
+			)
+		)
+	)
 	(global_label "SER_LATCH"
 		(shape input)
@@
 					(unit 1)
 				)
+			)
+		)
+	)
+	(symbol
+		(lib_id "power:PWR_FLAG")
+		(at 63.5 95.25 0)
+		(unit 1)
+		(exclude_from_sim no)
+		(in_bom yes)
+		(on_board yes)
+		(dnp no)
+		(fields_autoplaced yes)
+		(property "Reference" "#FLG02"
+			(at 63.5 93.345 0)
+			(effects
+				(font
+					(size 1.27 1.27)
+				)
+				(hide yes)
+			)
+		)
+		(property "Value" "PWR_FLAG"
+			(at 63.5 90.17 0)
+			(effects
+				(font
+					(size 1.27 1.27)
+				)
+			)
+		)
+		(property "Footprint" ""
+			(at 63.5 95.25 0)
+			(effects
+				(font
+					(size 1.27 1.27)
+				)
+				(hide yes)
+			)
+		)
+		(property "Datasheet" "~"
+			(at 63.5 95.25 0)
+			(effects
+				(font
+					(size 1.27 1.27)
+				)
+				(hide yes)
+			)
+		)
+		(property "Description" "Special symbol for telling ERC where power comes from"
+			(at 63.5 95.25 0)
+			(effects
+				(font
+					(size 1.27 1.27)
+				)
+				(hide yes)
+			)
+		)
+		(pin "1"
+		)
+		(instances
+			(project "schematic"
+				(path "/8bb2c8a8-35e3-4245-8e15-a816e35d5f01"
+					(reference "#FLG02")
+					(unit 1)
+				)
